File: kbtb/testdata/routed/numpad_board_routed.kicad_pcb (KiCad board)
At the start: 2 copper layers, 76.2 x 95.2 mm, 48 parts, among them J1 HRO-TYPE-C-31-M-12, J2 Tag-Connect_TC2030-IDC-FP_2x0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, SW0 SW_Cherry_MX_1.00u_PCB, SW1 SW_Cherry_MX_1.00u_PCB, SW10 SW_Cherry_MX_1.00u_PCB, SW11 SW_Cherry_MX_1.00u_PCB, SW12 SW_Cherry_MX_1.00u_PCB, SW13 SW_Cherry_MX_1.00u_PCB, SW14 SW_Cherry_MX_1.00u_PCB, SW15 SW_Cherry_MX_1.00u_PCB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

Commit message: Add support for Atmega32U4
Parts:
- C1, C2, C3: value 0.1 uF -> 0.1 µF
Changed lines of the file:
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@@
       (effects (font (size 1 1) (thickness 0.15)) (justify mirror))
     )
-    (fp_text value "0.1 uF" (at 0 -1.43) (layer "B.Fab")
+    (fp_text value "0.1 µF" (at 0 -1.43) (layer "B.Fab")
       (effects (font (size 1 1) (thickness 0.15)) (justify mirror))
     )
@@
       (effects (font (size 1 1) (thickness 0.15)) (justify mirror))
     )
-    (fp_text value "0.1 uF" (at 0 -1.43 270) (layer "B.Fab")
+    (fp_text value "0.1 µF" (at 0 -1.43 270) (layer "B.Fab")
       (effects (font (size 1 1) (thickness 0.15)) (justify mirror))
     )
@@
       (effects (font (size 1 1) (thickness 0.15)) (justify mirror))
     )
-    (fp_text value "0.1 uF" (at 0 -1.43 270) (layer "B.Fab")
-      (effects (font (size 1 1) (thickness 0.15)) (justify mirror))
-    )
+    (fp_text value "0.1 µF" (at 0 -1.43 270) (layer "B.Fab")
+      (effects (font (size 1 1) (thickness 0.15)) (justify mirror))
+    )
