File: examples/routed/numpad_board.kicad_pcb (KiCad board)
At the start: 2 copper layers, 76.2 x 95.2 mm, 53 parts, among them J1 HRO-TYPE-C-31-M-12, SW0 SW_Cherry_MX_1.00u_PCB, SW1 SW_Cherry_MX_1.00u_PCB, SW10 SW_Cherry_MX_1.00u_PCB, SW11 SW_Cherry_MX_1.00u_PCB, SW12 SW_Cherry_MX_1.00u_PCB, SW13 SW_Cherry_MX_1.00u_PCB, SW14 SW_Cherry_MX_1.00u_PCB, SW15 SW_Cherry_MX_1.00u_PCB, SW16 SW_Cherry_MX_1.00u_PCB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

Commit message: Add info text to PCB with fake hash
Other:
- board text added: "maude (a number pad) peterklein.dev"
Changed lines of the file:
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@@
   (gr_line (start 91.239842 16.10051) (end 91.274025 16.11418) (layer "Edge.Cuts") (width 0.1))
   (gr_line (start 17.389653 16.004064) (end 17.426398 16.001806) (layer "Edge.Cuts") (width 0.1))
+  (gr_text "maude (a number pad)\npeterklein.dev" (at 53.975 71.755) (layer "B.SilkS")
+    (effects (font (size 1.5 1.5) (thickness 0.3)) (justify mirror))
+  )
   (via (at 72.39 70.485) (size 0.8) (drill 0.4) (layers "F.Cu" "B.Cu") (free) (net 1))
   (via (at 58.42 51.435) (size 0.8) (drill 0.4) (layers "F.Cu" "B.Cu") (free) (net 1))
